File: hardware/kicad/xiamocon.kicad_pcb (KiCad board)
At the start: 2 copper layers, 100 x 50 mm, 103 parts, among them J1 JST S2B-PH-SM4-TB, J2 Conn_01x02, J3 Micro_SD_Card_Det_Hirose_DM3AT, J4 Hong Cheng HC-PM254-5.0H-2x10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, Q1 BSS138W, Q2 BSS138W, Q3 IRLML2246TRPBF, Q4 IRLML2246TRPBF, Q5 BSS138W, Q6 BSS138W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

Commit message: fix
Parts:
- added C17: 10u, Capacitor_SMD:C_0603_1608Metric, F.Cu at (135.4, 81.3)
- added D10: SP0502BAJT, Package_TO_SOT_SMD:SOT-323_SC-70, F.Cu at (97.1, 51.9)
- added D11: SP0502BAJT, Package_TO_SOT_SMD:SOT-323_SC-70, F.Cu at (95.8, 70.4)
- added D12: SP0502BAJT, Package_TO_SOT_SMD:SOT-323_SC-70, F.Cu at (104.9, 51.9)
- added D8: SP0502BAJT, Package_TO_SOT_SMD:SOT-323_SC-70, F.Cu at (85.1, 65.3)
- J4: value Hong Cheng HC-PM254-5.0H-2x10PS -> HC-PM254-5.0H-2x10PS
- moved J2 5.24 mm to (54.1, 68.1)
- moved R12 3.91 mm to (92.4, 52.3)
- moved FB2 3.07 mm to (59.2, 95.8), turned to 90 degrees
- moved C9 2.98 mm to (58.0, 79.2), turned to 180 degrees
- moved U4 2.87 mm to (56.6, 74.3)
- moved R22 2.80 mm to (55.1, 78.1)
- moved C15 2.79 mm to (53.7, 75.3)
- moved C8 2.79 mm to (53.2, 76.7)
- moved C12 2.54 mm to (59.2, 71.7)
- moved C16 2.54 mm to (59.5, 75.1)
- moved R43 2.54 mm to (60.6, 72.3)
- moved R44 2.54 mm to (59.4, 73.9)
- moved C11 2.43 mm to (57.9, 93.5)
- moved TP1 2.41 mm to (55.2, 80.4)
- moved C5 2.29 mm to (57.7, 87.1)
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Connections:
- net /IOEX_MUTE_N renamed /IOEX_MUTE
- net Net-(J4-Pin_12) renamed /EXT_SDA
- net Net-(J4-Pin_13) renamed /EXT_SCL
Routing:
- net Net-(R20-Pad2): track 15.8 -> 25.4 mm, vias 0 -> 1
- net /SPI_MOSI: track 69.5 -> 76.1 mm
- net /LCD_CS: track 80.0 -> 84.9 mm
- net GND: track 3.63 -> 6.92 mm, vias 199 -> 202
- net Net-(D4-A): track 24.8 -> 22.1 mm
- net VPERI: track 185.1 -> 187.6 mm
- net /EXT_SCL: track 8.96 -> 11.3 mm
- net VCOM: track 99.3 -> 97.2 mm
- net Net-(J2-Pin_2): track 11.6 -> 9.67 mm
- net /SPI_SCK: track 62.1 -> 64.1 mm
- net /LCD_DC: track 72.3 -> 74.2 mm
- net /EXT_SDA: track 17.8 -> 19.5 mm
- net Net-(U2-VIN): track 3.74 -> 5.32 mm
- net Net-(J2-Pin_1): track 7.69 -> 6.25 mm
- net /TFC_CS: track 47.0 -> 48.2 mm
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Other:
- outline, holes or cut-outs redrawn

Commit message: pcb rev2 checked
Parts:
- added D13: 1N4148WS, Diode_SMD:D_SOD-523, F.Cu at (135.7, 72.4)
- added D14: 1N4148WS, Diode_SMD:D_SOD-523, F.Cu at (135.7, 73.9)
- added G***: LOGO, LOGO, F.Cu at (117.5, 55.4)
- C16: value 1nF -> 1n
- D1, D2, D3, D4, D7: footprint Diode_SMD:D_SOD-323 -> Diode_SMD:D_SOD-523
- J1: value JST S2B-PH-SM4-TB -> FG PH-2AWT
- U7: footprint Package_TO_SOT_SMD:SOT-23-6 -> Package_TO_SOT_SMD:TSOT-23-6
- moved R5 3.05 mm to (133.3, 73.9), turned to 0 degrees
- moved R7 2.59 mm to (133.3, 72.6)
- moved Q2 2.47 mm to (130.5, 73.3)
- moved TP2 1.78 mm to (128.5, 71.1)
- moved D3 1.59 mm to (85.9, 55.3)
- moved J1 1.42 mm to (144.1, 63.1)
- moved Q5 1.19 mm to (69.8, 81.8)
- moved C1 1.16 mm to (84.2, 55.4)
- moved R4 1.03 mm to (143.6, 77.6)
- moved D2 0.71 mm to (143.6, 79.9)
- moved D1 0.50 mm to (84.6, 57.7)
- moved D4 0.39 mm to (73.0, 81.8)
- moved D7 0.38 mm to (80.1, 75.8)
Connections:
- R5 pad 2: /I2C_SCL -> Net-(D13-K)
Routing:
- net GND: track 6.92 -> 15.6 mm, vias 202 -> 206
- net /LCD_DC: track 74.2 -> 81.1 mm
- net Net-(U1-GP27): track 91.8 -> 88.7 mm
- net /XIAO_GPIO: track 67.0 -> 64.0 mm
- net /LCD_CS: track 84.9 -> 87.7 mm
- net Net-(D13-K): track 0.00 -> 2.67 mm
- net Net-(U1-BOOT): track 30.9 -> 33.5 mm
- net /+BAT: track 61.0 -> 63.5 mm
- net Net-(D1-A): track 12.9 -> 10.9 mm
- net +3V3: track 161.9 -> 160.0 mm
- net /PERI_EN_N: track 82.6 -> 80.8 mm
- net VANL: track 41.5 -> 43.3 mm
- net Net-(Q2-D): track 9.68 -> 8.31 mm
- net /SPI_MOSI: track 76.1 -> 77.1 mm
- net /SPI_MISO: track 58.0 -> 58.8 mm
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