File: hardware/kicad/xiamocon.kicad_pcb (KiCad board)
At the start: 2 copper layers, 100 x 50 mm, 111 parts, among them J1 FG PH-2AWT, J2 Conn_01x02, J3 Micro_SD_Card_Det_Hirose_DM3AT, J4 HC-PM254-5.0H-2x10PS, Q1 BSS138W, Q2 BSS138W, Q3 IRLML2246TRPBF, Q4 IRLML2246TRPBF, Q5 BSS138W, Q6 BSS138W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

Commit message: pcb rev.2 ordered
Parts:
- D10, D11, D12, D8: value SP0502BAJT -> TPD2E2U06DCKR
