File: hardware/kicad/xiamocon.kicad_sch (KiCad schematic)
At the start: 102 parts, among them J1 JST S2B-PH-SM4-TB, J2 Conn_01x02, J3 Micro_SD_Card_Det_Hirose_DM3AT, J4 Hong Cheng HC-PM254-5.0H-2x10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, Q1 BSS138W, Q2 BSS138W, Q3 IRLML2246TRPBF, Q4 IRLML2246TRPBF, Q5 BSS138W, Q6 BSS138W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

Commit message: fix
Parts:
- added C17: 10u, Capacitor_SMD:C_0603_1608Metric, symbol Device:C_Small
- added D10, D11, D12, D8: SP0502BAJT, Package_TO_SOT_SMD:SOT-323_SC-70, symbol Power_Protection:SP0502BAJT
- J4: value Hong Cheng HC-PM254-5.0H-2x10PS -> HC-PM254-5.0H-2x10PS
Connections:
- net EXT_AUDIO: now also D8.1 (K)
- net GND: now also C17.2, D10.3 (A), D11.3 (A), D12.3 (A), D8.3 (A)
- net LCD_CS: now also D10.1 (K)
- net LCD_DC: now also D10.2 (K)
- net SPI_MOSI: now also D12.1 (K)
- net SPI_SCK: now also D12.2 (K)
- net SPK_MUTE_N: now also D8.2 (K)
- net VPERI: now also C17.1
- net EXT_SDA: now reaches J4.12 (Pin_12), Q7.2 (S), R32.2, R34.1
- net EXT_SDA: now also D11.1 (K)
- net EXT_SCL: now reaches J4.13 (Pin_13), Q6.2 (S), R31.2, R33.2
- net EXT_SCL: now also D11.2 (K)
- net IOEX_MUTE_N renamed IOEX_MUTE
Other:
- note added: "Analog Power"
- note added: "Audio Power Amplifier and Speaker"
- note added: "Battery Voltage Monitoring"
- note added: "Display and TFCard"
- note added: "Extension Port"
- note added: "FUNC"
- note added: "IO Expander and Switches"
- note added: "MCU and Reset"
- note added: "Peripheral Power"
- note added: "X"
- note added: "Y"
- note removed: "MENU"
- note removed: "SELECT"
- note removed: "START"
- moved on the sheet: C10, C11, C12, C13, C14, C15, C16, C2, C3, C4, C5, C6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

Commit message: pcb rev2 checked
Parts:
- added D13, D14: 1N4148WS, Diode_SMD:D_SOD-523, symbol Device:D_Small
- C16: value 1nF -> 1n
- D1, D2, D3, D4, D7: footprint Diode_SMD:D_SOD-323 -> Diode_SMD:D_SOD-523; LCSC C60580 -> C917006; URL https://www.lcsc.com/product-detail/C60580.html -> https://www.lcsc.com/product-detail/C917006.html
- D10, D11, D12, D8: LCSC (none) -> C207262; URL (none) -> https://www.lcsc.com/product-detail/C207262.html
- J1: value JST S2B-PH-SM4-TB -> FG PH-2AWT; LCSC C295747 -> C2763693; URL https://www.lcsc.com/product-detail/C295747.html -> https://www.lcsc.com/product-detail/C2763693.html
- R7: LCSC C60491 -> C138033; URL https://www.lcsc.com/product-detail/C60491.html -> https://www.lcsc.com/product-detail/C138033.html
- U7: footprint Package_TO_SOT_SMD:SOT-23-6 -> Package_TO_SOT_SMD:TSOT-23-6; LCSC C2669855 -> C701590; URL https://www.lcsc.com/product-detail/C2669855.html -> https://www.lcsc.com/product-detail/C701590.html
Connections:
- net I2C_SCL: no longer R5.2
- net LCD_CS: now also D13.2 (A)
- net LCD_DC: now also D14.2 (A)
- new net: D13.1 (K), D14.1 (K), R5.2
Other:
- moved on the sheet: C2, C3, D5, Q2, Q3, R5, R6, R7, R8, TP2, TP6
