File: hardware/kicad/xiamocon.kicad_sch (KiCad schematic)
At the start: 109 parts, among them J1 FG PH-2AWT, J2 Conn_01x02, J3 Micro_SD_Card_Det_Hirose_DM3AT, J4 HC-PM254-5.0H-2x10PS, Q1 BSS138W, Q2 BSS138W, Q3 IRLML2246TRPBF, Q4 IRLML2246TRPBF, Q5 BSS138W, Q6 BSS138W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

Commit message: pcb rev.2 ordered
Parts:
- C1, C2, C5: LCSC C1705 -> C19666; URL https://www.lcsc.com/product-detail/C1705.html -> https://www.lcsc.com/product-detail/C19666.html
- C11, C3, C4: LCSC C14445 -> C52923; URL https://www.lcsc.com/product-detail/C14445.html -> https://www.lcsc.com/product-detail/C52923.html
- C12, C9: LCSC C140782 -> C15849; URL https://www.lcsc.com/product-detail/C140782.html -> https://www.lcsc.com/product-detail/C15849.html
- C16: LCSC C14442 -> C1523; URL https://www.lcsc.com/product-detail/C14442.html -> https://www.lcsc.com/product-detail/C1523.html
- D10, D11, D12, D8: value SP0502BAJT -> TPD2E2U06DCKR; LCSC C207262 -> C1855726; URL https://www.lcsc.com/product-detail/C207262.html -> https://www.lcsc.com/product-detail/C1855726.html
- D6: LCSC C60580 -> C2128; URL https://www.lcsc.com/product-detail/C60580.html -> https://www.lcsc.com/product-detail/C2128.html
- R1, R12, R13, R14, R15, R16, R17, R21, R37, R38, R8: LCSC C60490 -> C25744; URL https://www.lcsc.com/product-detail/C60490.html -> https://www.lcsc.com/product-detail/C25744.html
- R11, R22, R31, R32, R39, R40, R5, R6: LCSC C60491 -> C25741; URL https://www.lcsc.com/product-detail/C60491.html -> https://www.lcsc.com/product-detail/C25741.html
- R18, R19: LCSC C114762 -> C25879; URL https://www.lcsc.com/product-detail/C114762.html -> https://www.lcsc.com/product-detail/C25879.html
- R2, R9: LCSC C106232 -> C25076; URL https://www.lcsc.com/product-detail/C106232.html -> https://www.lcsc.com/product-detail/C25076.html
- R20, R23, R24, R25, R26, R27, R28, R33, R34, R35, R36: LCSC C106231 -> C17168; URL https://www.lcsc.com/product-detail/C106231.html -> https://www.lcsc.com/product-detail/C17168.html
- R29, R30: LCSC C105871 -> C25900; URL https://www.lcsc.com/product-detail/C105871.html -> https://www.lcsc.com/product-detail/C25900.html
- R4: LCSC C106235 -> C11702; URL https://www.lcsc.com/product-detail/C106235.html -> https://www.lcsc.com/product-detail/C11702.html
- R43, R44: LCSC C82868 -> C25768; URL https://www.lcsc.com/product-detail/C82868.html -> https://www.lcsc.com/product-detail/C25768.html
- R7: LCSC C138033 -> C26083; URL https://www.lcsc.com/product-detail/C138033.html -> https://www.lcsc.com/product-detail/C26083.html
